File: full-graphical/PCB/screen-driver/_autosave-screen-driver.kicad_sch (KiCad schematic)
At the start: 165 parts, among them J1 Barrel_Jack_Switch, J10 Conn_01x05_Male, J2 ANODE - EVEN 2-60, J3 ANODE - EVEN-62-100, J4 CATHODE - EVEN - 42-100, J5 CATHODE ODD 41-99, J6 CATHODE EVEN 2-40, J7 CATHODE ODD 1-39, J8 ANODE - ODD 1-59, J9 ANODE - ODD 61-99, Q1 MPSA42, Q10 MPSA42, Q11 MPSA42, Q12 MPSA42, Q13 MPSA42, Q14 MPSA42, Q15 MPSA42, Q16 MPSA42, Q17 MPSA42, Q18 MPSA42, Q19 MPSA42, Q2 MPSA42, Q20 MPSA42, Q21 MPSA42, Q22 MPSA42, Q23 MPSA42, Q24 MPSA42, Q25 MPSA42, Q26 MPSA42, Q27 MPSA42, Q28 MPSA42, Q29 MPSA42, Q3 MPSA42, Q30 MPSA42, Q31 MPSA42, Q32 MPSA42, Q4 MPSA42, Q5 MPSA42, Q6 MPSA42, Q7 MPSA42, Q8 MPSA42, Q9 MPSA42, U1 SN755870, U2 ESP32-DEVKIT-V1, U3 SN755870, U4 TSR_1-2450, U5 CD4017BE, U6 CD4017BE

Commit message: first draft of full pcb
Parts:
- gave numbers to parts that had none: 1
Connections:
- net GND: now also U1.32 (VDDH), U1.33 (VDDH), U1.35 (GND1), U1.36 (GND1), U1.37 (GND1), U1.40 (GND1), U1.41 (GND1), U1.43 (VDDH), U1.79 (VDDH), U1.80 (VDDH), U1.82 (GND1), U1.83 (GND1), U1.96 (VDDH), U1.97 (VDDH), U3.35 (GND1), U3.36 (GND1), U3.37 (GND1), U3.40 (GND1), U3.41 (GND1), U3.82 (GND1), U3.83 (GND1), U3.94 (GND1)
- net at U3.32 (VDDH): now also J10.3 (Pin_3), U1.44 (VDDH), U3.33 (VDDH), U3.43 (VDDH), U3.44 (VDDH), U3.79 (VDDH), U3.80 (VDDH), U3.96 (VDDH), U3.97 (VDDH)
