File: full-graphical/PCB/screen-driver/_autosave-screen-driver.kicad_sch (KiCad schematic)
At the start: 166 parts, among them J1 Barrel_Jack_Switch, J10 Conn_01x05_Male, J2 ANODE - EVEN 2-60, J3 ANODE - EVEN-62-100, J4 CATHODE - EVEN - 42-100, J5 CATHODE ODD 41-99, J6 CATHODE EVEN 2-40, J7 CATHODE ODD 1-39, J8 ANODE - ODD 1-59, J9 ANODE - ODD 61-99, Q1 MPSA42, Q10 MPSA42, Q11 MPSA42, Q12 MPSA42, Q13 MPSA42, Q14 MPSA42, Q15 MPSA42, Q16 MPSA42, Q17 MPSA42, Q18 MPSA42, Q19 MPSA42, Q2 MPSA42, Q20 MPSA42, Q21 MPSA42, Q22 MPSA42, Q23 MPSA42, Q24 MPSA42, Q25 MPSA42, Q26 MPSA42, Q27 MPSA42, Q28 MPSA42, Q29 MPSA42, Q3 MPSA42, Q30 MPSA42, Q31 MPSA42, Q32 MPSA42, Q4 MPSA42, Q5 MPSA42, Q6 MPSA42, Q7 MPSA42, Q8 MPSA42, Q9 MPSA42, U1 SN755870, U2 ESP32-DEVKITC-32D, U3 SN755870, U4 TSR_1-2450, U5 CD4017BE, U6 CD4017BE

Commit message: fixed footprint error in pcb and improved ground traces
Parts:
- gave numbers to parts that had none: 1
Changed lines of the file:
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@@
   (symbol (lib_id "Connector_Generic:Conn_01x04") (at 369.57 68.58 0) (unit 1)
     (in_bom yes) (on_board yes) (fields_autoplaced)
-    (property "Reference" "J?" (id 0) (at 372.11 68.5799 0)
+    (property "Reference" "J11" (id 0) (at 372.11 68.5799 0)
       (effects (font (size 1.27 1.27)) (justify left))
     )
@@
     )
     (path "/4aca60e3-f8df-4367-8b12-a8182ed36464"
-      (reference "J?") (unit 1) (value "Conn_01x04") (footprint "Connector_PinSocket_2.54mm:PinSocket_1x04_P2.54mm_Vertical")
+      (reference "J11") (unit 1) (value "Conn_01x04") (footprint "Connector_PinSocket_2.54mm:PinSocket_1x04_P2.54mm_Vertical")
     )
     (path "/859f3a46-66b3-4c1d-837a-8a588a31914b"
