File: full-graphical/PCB/screen-driver/screen-driver.kicad_sch (KiCad schematic)
At the start: 166 parts, among them J1 Barrel_Jack_Switch, J10 Conn_01x05_Male, J2 ANODE - EVEN 2-60, J3 ANODE - EVEN-62-100, J4 CATHODE - EVEN - 42-100, J5 CATHODE ODD 41-99, J6 CATHODE EVEN 2-40, J7 CATHODE ODD 1-39, J8 ANODE - ODD 1-59, J9 ANODE - ODD 61-99, Q1 MPSA42, Q10 MPSA42, Q11 MPSA42, Q12 MPSA42, Q13 MPSA42, Q14 MPSA42, Q15 MPSA42, Q16 MPSA42, Q17 MPSA42, Q18 MPSA42, Q19 MPSA42, Q2 MPSA42, Q20 MPSA42, Q21 MPSA42, Q22 MPSA42, Q23 MPSA42, Q24 MPSA42, Q25 MPSA42, Q26 MPSA42, Q27 MPSA42, Q28 MPSA42, Q29 MPSA42, Q3 MPSA42, Q30 MPSA42, Q31 MPSA42, Q32 MPSA42, Q4 MPSA42, Q5 MPSA42, Q6 MPSA42, Q7 MPSA42, Q8 MPSA42, Q9 MPSA42, U1 SN755870, U2 ESP32-DEVKITC-32D, U3 SN755870, U4 TSR_1-2450, U5 CD4017BE, U6 CD4017BE

Commit message: added rev3 PCB
Parts:
- removed J?: Conn_01x04, symbol Connector_Generic:Conn_01x04
- removed U1, U3: SN755870, Package_QFP:TQFP-100_14x14mm_P0.5mm, symbol sn755870:SN755870
- removed U2: ESP32-DEVKITC-32D, MODULE_ESP32-DEVKITC-32D, symbol ESP32-DEVKITC-32D:ESP32-DEVKITC-32D
- added C5, C6: C_Small, Capacitor_THT:C_Disc_D3.8mm_W2.6mm_P2.50mm, symbol Device:C_Small
- added Q33: BC547, Package_TO_SOT_THT:TO-92_Inline, symbol Transistor_BJT:BC547
- added R114, R115, R116: 330, Resistor_THT:R_Axial_DIN0207_L6.3mm_D2.5mm_P10.16mm_Horizontal, symbol Device:R
- added R117: 10k, Resistor_THT:R_Axial_DIN0207_L6.3mm_D2.5mm_P10.16mm_Horizontal, symbol Device:R
- added R118: 100, Resistor_THT:R_Axial_DIN0207_L6.3mm_D2.5mm_P10.16mm_Horizontal, symbol Device:R
- added R119, R120, R121, R122, R123, R124, R125, R126, R127, R128, R129, R130, R131, R132, R133, R134, R135, R136, R137, R138, R139, R140, R141, R142, R143, R144, R145, R146, R147, R148, R149, R150, R151, R152, R153, R154, R155, R156, R157, R158, R159, R160, R161, R162, R163, R164, R165, R166, R167, R168: 330k, Resistor_THT:R_Axial_DIN0207_L6.3mm_D2.5mm_P10.16mm_Horizontal, symbol Device:R
- added R169, R170, R171, R172, R173, R174, R175, R176, R177, R178, R179, R180, R181, R182, R183, R184, R185, R186, R187, R188, R189, R190, R191, R192, R193, R194, R195, R196, R197, R198, R199, R200, R201, R202, R203, R204, R205, R206, R207, R208, R209, R210, R211, R212, R213, R214, R215, R216, R217, R218: 390k, Resistor_THT:R_Axial_DIN0207_L6.3mm_D2.5mm_P10.16mm_Horizontal, symbol Device:R
- added RV1: R_Potentiometer, symbol Device:R_Potentiometer
- added U1: SC0915, MODULE_SC0915, symbol SC0915:SC0915
- added U10: level_converter, daughter_boards:level_shifter, symbol daughter_boards:level_converter
- added U11, U7, U8: YH5504KH01, soviet:YH5504KH01, symbol soviet:YH5504KH01
- added U12, U13, U2, U3: TLP627, Package_DIP:DIP-4_W7.62mm, symbol Isolator:TLP627
- added U9: 74HC595, Package_DIP:DIP-16_W7.62mm, symbol 74xx:74HC595
- R1, R10, R11, R12, R13, R14, R15, R16, R17, R18, R19, R2, R20, R21, R22, R23, R24, R25, R26, R27, R28, R29, R3, R30, R31, R32, R33, R34, R35, R36, R37, R38, R39, R4, R40, R41, R42, R43, R44, R45, R46, R47, R48, R49, R5, R50, R6, R7, R8, R9: value R -> 390k; footprint Resistor_SMD:R_0201_0603Metric_Pad0.64x0.40mm_HandSolder -> Resistor_THT:R_Axial_DIN0207_L6.3mm_D2.5mm_P10.16mm_Horizontal
- R100, R102, R103, R104, R105, R106, R107, R108, R109, R110, R111, R61, R62, R63, R64, R65, R66, R67, R68, R69, R70, R71, R72, R73, R74, R75, R76, R77, R78, R79, R80, R81, R82, R83, R84, R85, R86, R87, R88, R89, R90, R91, R92, R93, R94, R95, R96, R97, R98, R99: value R -> 330k; footprint Resistor_SMD:R_0201_0603Metric_Pad0.64x0.40mm_HandSolder -> Resistor_THT:R_Axial_DIN0207_L6.3mm_D2.5mm_P10.16mm_Horizontal
- R113: value R -> 330; footprint Resistor_THT:R_Axial_DIN0207_L6.3mm_D2.5mm_P7.62mm_Horizontal -> Resistor_THT:R_Axial_DIN0207_L6.3mm_D2.5mm_P10.16mm_Horizontal
Connections:
- net +3V3: now also U1.36 (3V3_OUT), U10.3 (LV_in); no longer C2.1, C3.1
- net +5V: now also C2.1, C3.1, C5.1, C6.1, R118.1, U10.10 (HV_in), U11.4 (VCC), U11.42 (VCC), U7.4 (VCC), U7.42 (VCC), U8.4 (VCC), U8.42 (VCC), U9.10 (~{SRCLR}), U9.16 (VCC)
- net GND: now also C5.2, C6.2, Q33.3 (E), RV1.2, U1.13 (GND), U1.18 (GND), U1.23 (GND), U1.28 (GND), U1.3 (GND), U1.38 (GND), U1.8 (GND), U1.D2 (GND), U10.4 (GND), U10.9 (GND), U11.21 (gnd), U11.39 (gnd), U11.5 (gnd), U12.2, U12.3, U13.2, U13.3, U2.2, U2.3, U3.2, U3.3, U7.21 (gnd), U7.39 (gnd), U7.5 (gnd), U8.21 (gnd), U8.39 (gnd), U8.5 (gnd), U9.13 (~{OE}), U9.8 (GND); no longer R113.2
- net at J9.6 (Pin_6): now also R158.1, R208.2; no longer R100.1
- net at R100.2: now also U11.22 (OUT16)
- net at R37.1: now also J10.3 (Pin_3), R1.1, R10.1, R11.1, R12.1, R13.1, R14.1, R15.1, R16.1, R17.1, R18.1, R19.1, R2.1, R20.1, R21.1, R22.1, R23.1, R24.1, R25.1, R26.1, R27.1, R28.1, R29.1, R3.1, R30.1, R31.1, R32.1, R33.1, R34.1, R35.1, R36.1, R38.1, R39.1, R4.1, R40.1, R41.1, R42.1, R43.1, R44.1, R45.1, R46.1, R47.1, R48.1, R49.1, R5.1, R50.1, R6.1, R7.1, R8.1, R9.1, R169.1, R170.1, R171.1, R172.1, R173.1, R174.1, R175.1, R176.1, R177.1, R178.1, R179.1, R180.1, R181.1, R182.1, R183.1, R184.1, R185.1, R186.1, R187.1, R188.1, R189.1, R190.1, R191.1, R192.1, R193.1, R194.1, R195.1, R196.1, R197.1, R198.1, R199.1, R200.1, R201.1, R202.1, R203.1, R204.1, R205.1, R206.1, R207.1, R208.1, R209.1, R210.1, R211.1, R212.1, R213.1, R214.1, R215.1, R216.1, R217.1, R218.1; no longer J3.3 (Pin_3)
- net at R37.2: now also J2.25 (Pin_25), R97.1
- net at J3.14 (Pin_14): now also R14.2, R74.1; no longer R48.1
- net at R48.2: now also J2.38 (Pin_38), R109.1
- net at J9.11 (Pin_11): now also R163.1, R213.2; no longer R106.1
- net at R106.2: now also U11.32 (OUT26)
- net at J2.26 (Pin_26): now also R38.2, R98.1; no longer R22.1
- net at R22.2: now also J2.10 (Pin_10), R82.1
- net at R65.1: now also J3.5 (Pin_5), R5.2; no longer J8.9 (Pin_9)
- net at R65.2: now also U8.19 (OUT14)
- net at J8.15 (Pin_15): now also R129.1, R179.2; no longer R71.1
- net at R71.2: now also U8.32 (OUT26)
- net at R63.2: now also U8.15 (OUT10)
- net at R72.2: now also U8.34 (OUT28)
- net at R62.2: now also U8.13 (OUT8)
- net at R73.2: now also U8.36 (OUT30)
- net at R74.2: now also U8.38 (OUT32)
- net at R75.2: now also U3.4
- net at R76.2: now also U2.4
- net at R77.2: now also U7.7 (OUT2)
- net at R78.2: now also U7.9 (OUT4)
- net at R79.2: now also U7.11 (OUT6)
- net at R80.2: now also U7.13 (OUT8)
- net at R81.2: now also U7.15 (OUT10)
- net at R64.2: now also U8.17 (OUT12)
- net at R82.2: now also U7.17 (OUT12)
- net at R83.2: now also U7.19 (OUT14)
- net at R84.2: now also U7.22 (OUT16)
- net at R85.2: now also U7.24 (OUT18)
- net at R86.2: now also U7.26 (OUT20)
- net at R87.2: now also U7.28 (OUT22)
- net at R88.2: now also U7.30 (OUT24)
- net at R89.2: now also U7.32 (OUT26)
- net at R90.2: now also U7.34 (OUT28)
- net at R91.2: now also U7.36 (OUT30)
- net at R92.2: now also U7.38 (OUT32)
- net at R66.2: now also U8.22 (OUT16)
- net at R93.2: now also U11.7 (OUT2)
- net at R94.2: now also U11.9 (OUT4)
- net at R95.2: now also U11.11 (OUT6)
- net at R96.2: now also U11.13 (OUT8)
- net at R67.2: now also U8.24 (OUT18)
- net at R97.2: now also U11.15 (OUT10)
- net at R98.2: now also U11.17 (OUT12)
- net at R99.2: now also U11.19 (OUT14)
- net at R102.2: now also U11.24 (OUT18)
- net at R103.2: now also U11.26 (OUT20)
- net at R104.2: now also U11.28 (OUT22)
- net at R105.2: now also U11.30 (OUT24)
- net at R107.2: now also U11.34 (OUT28)
- net at R68.2: now also U8.26 (OUT20)
- net at R108.2: now also U11.36 (OUT30)
- net at R109.2: now also U11.38 (OUT32)
- net at R110.2: now also U8.7 (OUT2)
- net at R111.2: now also U8.9 (OUT4)
- net at R69.2: now also U8.28 (OUT22)
- net at R70.2: now also U8.30 (OUT24)
- net at R61.2: now also U8.11 (OUT6)
- net at J9.4 (Pin_4): now also R156.1, R206.2; no longer R98.1
- net at R108.1: now also J2.37 (Pin_37), R47.2; no longer J9.13 (Pin_13)
- net at J2.21 (Pin_21): now also R33.2, R93.1; no longer R17.1
- net at R17.2: now also J2.5 (Pin_5), R77.1
- net at J3.15 (Pin_15): now also R15.2, R75.1; no longer R49.1
- net at R49.2: now also J2.39 (Pin_39), R110.1
- net at R95.1: now also J2.23 (Pin_23), R35.2; no longer J9.1 (Pin_1)
- net at J9.10 (Pin_10): now also R162.1, R212.2; no longer R105.1
- net at J9.12 (Pin_12): now also R164.1, R214.2; no longer R107.1
- net at J9.14 (Pin_14): now also R166.1, R216.2; no longer R109.1
- net at J9.15 (Pin_15): now also R167.1, R217.2; no longer R110.1
- net at J9.16 (Pin_16): now also R168.1, R218.2; no longer R111.1
- net at R96.1: now also J2.24 (Pin_24), R36.2; no longer J9.2 (Pin_2)
- net at J9.3 (Pin_3): now also R155.1, R205.2; no longer R97.1
- net at R99.1: now also J2.27 (Pin_27), R39.2; no longer J9.5 (Pin_5)
- net at J9.7 (Pin_7): now also R159.1, R209.2; no longer R102.1
- net at J9.8 (Pin_8): now also R160.1, R210.2; no longer R103.1
- net at R104.1: now also J2.33 (Pin_33), R43.2; no longer J9.9 (Pin_9)
- net at J2.19 (Pin_19): now also R31.2, R91.1; no longer R15.1
- net at U5.14 (CLOCK): now also U1.6 (GP4)
- net at U5.15 (RESET): now also U1.5 (GP3)
- net at R27.2: now also J2.15 (Pin_15), R87.1
- net at R88.1: now also J2.16 (Pin_16), R28.2; no longer J8.34 (Pin_34)
- net at U6.15 (RESET): now also U1.7 (GP5)
- net at U6.14 (CLOCK): now also U1.9 (GP6)
- net at J8.23 (Pin_23): now also R137.1, R187.2; no longer R79.1
- net at J3.7 (Pin_7): now also R67.1, R7.2; no longer R41.1
- net at R41.2: now also J2.29 (Pin_29), R102.1
- net at J2.11 (Pin_11): now also R23.2, R83.1; no longer R7.1
- net at J2.28 (Pin_28): now also R100.1, R40.2; no longer R24.1
- net at R24.2: now also J2.12 (Pin_12), R84.1
- net at J8.26 (Pin_26): now also R140.1, R190.2; no longer R82.1
- net at J3.1 (Pin_1): now also R1.2, R61.1; no longer R35.1
- net at J8.11 (Pin_11): now also R125.1, R175.2; no longer R67.1
- net at R12.2: now also J3.12 (Pin_12), R72.1
- net at R8.2: now also J3.8 (Pin_8), R68.1
- net at J8.33 (Pin_33): now also R145.1, R195.2; no longer R87.1
- net at J2.6 (Pin_6): now also R18.2, R78.1; no longer R2.1
- net at R2.2: now also J3.2 (Pin_2), R62.1
- net at J8.27 (Pin_27): now also R141.1, R191.2; no longer R83.1
- net at J2.40 (Pin_40): now also R111.1, R50.2; no longer R34.1
- net at R34.2: now also J2.22 (Pin_22), R94.1
- net at R21.2: now also J2.9 (Pin_9), R81.1
- net at J2.18 (Pin_18): now also R30.2, R90.1; no longer R14.1
- net at J2.34 (Pin_34): now also R105.1, R44.2; no longer R28.1
- net at J8.38 (Pin_38): now also R150.1, R200.2; no longer R92.1
- net at J8.16 (Pin_16): now also R130.1, R180.2; no longer R72.1
- net at R63.1: now also J3.3 (Pin_3), R3.2; no longer J8.7 (Pin_7)
- net at J2.35 (Pin_35): now also R106.1, R45.2; no longer R29.1
- net at R29.2: now also J2.17 (Pin_17), R89.1
- net at J2.7 (Pin_7): now also R19.2, R79.1; no longer R3.1
- net at J8.19 (Pin_19): now also R133.1, R183.2; no longer R75.1
- net at J2.13 (Pin_13): now also R25.2, R85.1; no longer R9.1
- net at J2.14 (Pin_14): now also R26.2, R86.1; no longer R10.1
- net at J2.20 (Pin_20): now also R32.2, R92.1; no longer R16.1
- net at J2.32 (Pin_32): now also R103.1, R42.2; no longer R26.1
- net at J2.36 (Pin_36): now also R107.1, R46.2; no longer R30.1
- net at J2.8 (Pin_8): now also R20.2, R80.1; no longer R4.1
- net at R10.2: now also J3.10 (Pin_10), R70.1
- net at R13.2: now also J3.13 (Pin_13), R73.1
- net at R4.2: now also J3.4 (Pin_4), R64.1
- net at R9.2: now also J3.9 (Pin_9), R69.1
- net at J8.5 (Pin_5): now also R119.1, R169.2; no longer R61.1
- net at R16.2: now also J3.16 (Pin_16), R76.1
- net at R6.2: now also J3.6 (Pin_6), R66.1
- net at R11.2: now also J3.11 (Pin_11), R71.1
- net at J8.40 (Pin_40): now also R152.1, R202.2; no longer R94.1
- net at J8.6 (Pin_6): now also R120.1, R170.2; no longer R62.1
- net at J8.20 (Pin_20): now also R134.1, R184.2; no longer R76.1
- net at J10.4 (Pin_4): now also RV1.1; no longer R113.1
- net at J8.21 (Pin_21): now also R135.1, R185.2; no longer R77.1
- net at J8.10 (Pin_10): now also R124.1, R174.2; no longer R66.1
- net at J8.29 (Pin_29): now also R143.1, R193.2; no longer R85.1
- net at J8.32 (Pin_32): now also R144.1, R194.2; no longer R86.1
- net at J8.13 (Pin_13): now also R127.1, R177.2; no longer R69.1
- net at J8.22 (Pin_22): now also R136.1, R186.2; no longer R78.1
- net at J8.35 (Pin_35): now also R147.1, R197.2; no longer R89.1
- net at J8.36 (Pin_36): now also R148.1, R198.2; no longer R90.1
- net at J8.25 (Pin_25): now also R139.1, R189.2; no longer R81.1
- net at J8.14 (Pin_14): now also R128.1, R178.2; no longer R70.1
- net at J8.28 (Pin_28): now also R142.1, R192.2; no longer R84.1
- net at J8.24 (Pin_24): now also R138.1, R188.2; no longer R80.1
- net at J8.18 (Pin_18): now also R132.1, R182.2; no longer R74.1
- net at J8.12 (Pin_12): now also R126.1, R176.2; no longer R68.1
- net at J8.17 (Pin_17): now also R131.1, R181.2; no longer R73.1
- net at J8.37 (Pin_37): now also R149.1, R199.2; no longer R91.1
- net at J8.39 (Pin_39): now also R151.1, R201.2; no longer R93.1
- net at J8.8 (Pin_8): now also R122.1, R172.2; no longer R64.1
- new net: R114.1, U3.1
- new net: R139.2, U11.14 (OUT9)
- new net: Q33.1 (C), R118.2, U11.3 (~latch), U7.3 (~latch), U8.3 (~latch)
- new net: R124.2, U7.16 (OUT11)
- new net: J9.13 (Pin_13), R165.1, R215.2
- new net: R142.2, U11.20 (OUT15)
- new net: U10.12 (HV1), U7.1 (SER_IN)
- new net: R121.2, U7.10 (OUT5)
- new net: R122.2, U7.12 (OUT7)
- new net: R123.2, U7.14 (OUT9)
- new net: R125.2, U7.18 (OUT13)
- new net: R126.2, U7.20 (OUT15)
- new net: R127.2, U7.23 (OUT17)
- new net: R128.2, U7.25 (OUT19)
- new net: R129.2, U7.27 (OUT21)
- new net: R130.2, U7.29 (OUT23)
- new net: R131.2, U7.31 (OUT25)
- new net: R132.2, U7.33 (OUT27)
- new net: R133.2, U7.35 (OUT29)
- new net: R134.2, U7.37 (OUT31)
- new net: R117.1, U10.11 (HV2), U11.40 (latch), U7.40 (latch), U8.40 (latch), U9.12 (RCLK)
- new net: U11.1 (SER_IN), U7.41 (SER_OUT)
- new net: R119.2, U7.6 (OUT1)
- new net: R120.2, U7.8 (OUT3)
- new net: R148.2, U11.33 (OUT27)
- new net: R166.2, U8.37 (OUT31)
- new net: J9.1 (Pin_1), R153.1, R203.2
- new net: R140.2, U11.16 (OUT11)
- new net: R147.2, U11.31 (OUT25)
- new net: R159.2, U8.23 (OUT17)
- new net: R116.1, U13.1
- new net: R168.2, U13.4
- new net: J9.2 (Pin_2), R154.1, R204.2
- new net: J9.5 (Pin_5), R157.1, R207.2
- new net: J9.9 (Pin_9), R161.1, R211.2
- new net: U1.1 (GP0), U10.1 (LV1)
- new net: U1.2 (GP1), U10.2 (LV2)
- new net: U1.4 (GP2), U10.5 (LV3)
- new net: R161.2, U8.27 (OUT21)
- new net: R156.2, U8.16 (OUT11)
- new net: R157.2, U8.18 (OUT13)
- new net: J8.34 (Pin_34), R146.1, R196.2
- new net: R146.2, U11.29 (OUT23)
- new net: R165.2, U8.35 (OUT29)
- new net: R164.2, U8.33 (OUT27)
- new net: R145.2, U11.27 (OUT21)
- new net: R153.2, U8.10 (OUT5)
- new net: R162.2, U8.29 (OUT23)
- new net: R115.1, U12.1
- new net: R115.2, U9.15 (QA)
- new net: R137.2, U11.10 (OUT5)
- new net: R138.2, U11.12 (OUT7)
- new net: R141.2, U11.18 (OUT13)
- new net: R143.2, U11.23 (OUT17)
- new net: R144.2, U11.25 (OUT19)
- new net: R149.2, U11.35 (OUT29)
- new net: R150.2, U11.37 (OUT31)
- new net: U11.41 (SER_OUT), U8.1 (SER_IN)
- new net: R135.2, U11.6 (OUT1)
- new net: R136.2, U11.8 (OUT3)
- new net: R116.2, U9.2 (QC)
- new net: R167.2, U12.4
- new net: R114.2, U9.1 (QB)
- new net: R152.2, U8.8 (OUT3)
- new net: R155.2, U8.14 (OUT9)
- new net: J8.9 (Pin_9), R123.1, R173.2
- new net: R158.2, U8.20 (OUT15)
- new net: R163.2, U8.31 (OUT25)
- new net: R160.2, U8.25 (OUT19)
- new net: Q33.2 (B), R117.2
- new net: R113.2, U2.1
- new net: R151.2, U8.6 (OUT1)
- new net: R154.2, U8.12 (OUT7)
- new net: J8.7 (Pin_7), R121.1, R171.2
- new net: U8.41 (SER_OUT), U9.14 (SER)
- new net: R113.1, U9.3 (QD)
- new net: U1.A (USB_SHIELD), U1.B (USB_SHIELD), U1.C (USB_SHIELD), U1.D (USB_SHIELD)
- new net clk: U10.8 (HV3), U11.2 (clk), U7.2 (clk), U8.2 (clk), U9.11 (SRCLK)
Other:
- note added: "TODO: Check everything"
